Commit message: works with moveit and gazebo. before refactoring

File: so101_description/urdf/so101_new_calib.ros2_control.xacro (robot description, xacro)
@@ -2,13 +2,22 @@
 <robot xmlns:xacro="http://www.ros.org/wiki/xacro" name="so101_new_calib">
     <xacro:macro name="so101_new_calib_ros2_control" params="name initial_positions_file">
-        <xacro:property name="initial_positions" value="${load_yaml(initial_positions_file)['initial_positions']}"/>
+        <xacro:property name="initial_positions" value="${xacro.load_yaml(initial_positions_file)['initial_positions']}"/>
         <ros2_control name="${name}" type="system">
-            <hardware>
-                <!-- By default, set up controllers for simulation. This won't work on real hardware -->
-                <!-- plugin>mock_components/GenericSystem</plugin -->
-                <plugin>topic_based_ros2_control/TopicBasedSystem</plugin>
-                <param name="joint_commands_topic">/isaac_joint_command</param>
-                <param name="joint_states_topic">/isaac_joint_states</param>
-            </hardware>
+          <hardware>
+            <!-- plugin> mock_components/GenericSystem </plugin -->
+            <xacro:if value="$(eval mode == 'isaac')">
+              <plugin>topic_based_ros2_control/TopicBasedSystem</plugin>
+              <param name="joint_commands_topic">/isaac_joint_command</param>
+              <param name="joint_states_topic">/isaac_joint_states</param>
+            </xacro:if>
+            <!-- <xacro:if value="$(eval mode == 'gazebo')"> -->
+            <plugin>ign_ros2_control/IgnitionSystem</plugin>
+            <!-- </xacro:if> -->
+            <xacro:if value="$(eval mode == 'real')">
+              <plugin>so101_hardware/So101System</plugin>
+              <param name="serial_port">/dev/ttyUSB0</param>
+              <param name="baudrate">115200</param>
+            </xacro:if>
+          </hardware>
             <joint name="Rotation">
                 <command_interface name="position"/>

File: so101_description/urdf/so101_new_calib.urdf (robot description, URDF)
Before this commit: robot so101_new_calib, 7 links, 6 joints
Links:
- added link world
Joints:
- added joint world_to_base: type fixed, parent world, child base, origin xyz=0 0 0 rpy=0 0 0

File: so101_description/urdf/so101_new_calib.urdf.xacro (robot description, xacro)
@@ -4,12 +4,15 @@
     <xacro:arg name="initial_positions_file" default="$(find so101_description)/config/initial_positions.yaml" />
     <xacro:arg name="display" default="false"/>
+    <xacro:arg name="mode" default="gazebo"/>
+    <!-- or 'isaac' or 'real' -->
     <!-- Import so101_new_calib urdf file -->
     <xacro:include filename="$(find so101_description)/urdf/so101_new_calib.urdf" />
     <!-- Conditionally include transmissions & control -->
     <xacro:if value="$(eval not display)">
+        <xacro:include filename="$(find so101_description)/urdf/so101_new_calib_gazebo.xacro"/>
         <xacro:include filename="$(find so101_description)/urdf/so101_new_calib_with_transmission.xacro"/>
-        <!-- Import control_xacro -->
-        <xacro:include filename="so101_new_calib.ros2_control.xacro" />
-        <xacro:so101_new_calib_ros2_control name="FakeSystem" initial_positions_file="$(arg initial_positions_file)"/>
+            <!-- Import control_xacro -->
+        <xacro:include filename="$(find so101_description)/urdf/so101_new_calib.ros2_control.xacro" />
+        <xacro:so101_new_calib_ros2_control name="RobotSystem" initial_positions_file="$(arg initial_positions_file)"/>
     </xacro:if>
 </robot>

File: so101_description/urdf/so101_new_calib_with_transmission.xacro (robot description, xacro)
@@ -1,4 +1,4 @@
 <?xml version="1.0"?>
-<robot xmlns:xacro="http://ros.org/wiki/xacro">
+<robot xmlns:xacro="http://ros.org/wiki/xacro" name="so101_new_calib">
     <transmission name="6_trans">
         <type>transmission_interface/SimpleTransmission</type>

Commit message: update

File: so101_description/urdf/so101_new_calib.ros2_control.xacro (robot description, xacro)
@@ -20,43 +20,43 @@
             </xacro:if>
           </hardware>
-            <joint name="Rotation">
+            <joint name="shoulder_pan">
                 <command_interface name="position"/>
                 <state_interface name="position">
-                  <param name="initial_value">${initial_positions['Rotation']}</param>
+                  <param name="initial_value">${initial_positions['shoulder_pan']}</param>
                 </state_interface>
                 <state_interface name="velocity"/>
             </joint>
-            <joint name="Pitch">
+            <joint name="shoulder_lift">
                 <command_interface name="position"/>
                 <state_interface name="position">
-                  <param name="initial_value">${initial_positions['Pitch']}</param>
+                  <param name="initial_value">${initial_positions['shoulder_lift']}</param>
                 </state_interface>
                 <state_interface name="velocity"/>
             </joint>
-            <joint name="Elbow">
+            <joint name="elbow_flex">
                 <command_interface name="position"/>
                 <state_interface name="position">
-                  <param name="initial_value">${initial_positions['Elbow']}</param>
+                  <param name="initial_value">${initial_positions['elbow_flex']}</param>
                 </state_interface>
                 <state_interface name="velocity"/>
             </joint>
-            <joint name="Wrist_Pitch">
+            <joint name="wrist_flex">
                 <command_interface name="position"/>
                 <state_interface name="position">
-                  <param name="initial_value">${initial_positions['Wrist_Pitch']}</param>
+                  <param name="initial_value">${initial_positions['wrist_flex']}</param>
                 </state_interface>
                 <state_interface name="velocity"/>
             </joint>
-            <joint name="Wrist_Roll">
+            <joint name="wrist_roll">
                 <command_interface name="position"/>
                 <state_interface name="position">
-                  <param name="initial_value">${initial_positions['Wrist_Roll']}</param>
+                  <param name="initial_value">${initial_positions['wrist_roll']}</param>
                 </state_interface>
                 <state_interface name="velocity"/>
             </joint>
-            <joint name="Jaw">
+            <joint name="gripper">
                 <command_interface name="position"/>
                 <state_interface name="position">
-                  <param name="initial_value">${initial_positions['Jaw']}</param>
+                  <param name="initial_value">${initial_positions['gripper']}</param>
                 </state_interface>
                 <state_interface name="velocity"/>

File: so101_description/urdf/so101_new_calib1.urdf (robot description, URDF)
Before this commit: robot so101_new_calib, 9 links, 8 joints
Links:
- removed link base_link
- removed link gripper_frame_link
- removed link gripper_link
- removed link lower_arm_link
- removed link moving_jaw_so101_v1_link
- removed link shoulder_link
- removed link upper_arm_link
- removed link wrist_link
- added link base, mass 0.147; collision mesh filename=package://so101_description/meshes/base_motor_holder_so101_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; collision mesh filename=package://so101_description/meshes/base_so101_v2.stl
- added link gripper, mass 0.087; collision mesh filename=package://so101_description/meshes/sts3215_03a_v1.stl; collision mesh filename=package://so101_description/meshes/wrist_roll_follower_so10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
- added link jaw, mass 0.012; collision mesh filename=package://so101_description/meshes/moving_jaw_so101_v1.stl; visual mesh filename=package://so101_description/meshes/moving_jaw_so101_v1.stl
- added link lower_arm, mass 0.104; collision mesh filename=package://so101_description/meshes/motor_holder_so101_wrist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; collision mesh filename=package://so101_description/meshes/sts3215_03a_v1.stl
- added link shoulder, mass 0.100006; collision mesh filename=package://so101_description/meshes/motor_holder_so101_base_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; collision mesh filename=package://so101_description/meshes/rotation_pitch_so101_v1.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
- added link upper_arm, mass 0.103; collision mesh filename=package://so101_description/meshes/sts3215_03a_v1.stl; collision mesh filename=package://so101_description/meshes/upper_arm_so101_v1.stl
- added link wrist, mass 0.079; collision mesh filename=package://so101_description/meshes/sts3215_03a_no_horn_v1.s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; collision mesh filename=package://so101_description/meshes/wrist_roll_pitch_so101_v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
Joints:
- removed joint elbow_flex
- removed joint gripper
- removed joint gripper_frame_joint
- removed joint shoulder_lift
- removed joint shoulder_pan
- removed joint wrist_flex
- removed joint wrist_roll
- added joint Elbow: type revolute, parent upper_arm, child lower_arm, origin xyz=-0.11257 -0.028 2.46331e-16 rpy=-1.22818e-15 5.75928e-16 1.5708, axis 0 0 1, limit lower=-1.74533 upper=1.5708 effort=10 velocity=10
- added joint Jaw: type revolute, parent gripper, child jaw, origin xyz=0.0202 0.0188 -0.0234 rpy=1.5708 -5.14108e-17 -1.38655e-14, axis 0 0 1, limit lower=-0.174533 upper=1.74533 effort=10 velocity=10
- added joint Pitch: type revolute, parent shoulder, child upper_arm, origin xyz=-0.0303992 -0.0182778 -0.0542 rpy=-1.5708 -1.5708 0, axis 0 0 1, limit lower=-1.74533 upper=1.74533 effort=10 velocity=10
- added joint Rotation: type revolute, parent base, child shoulder, origin xyz=0.0207909 -0.0230745 0.0948817 rpy=-3.14159 6.03684e-16 1.5708, axis 0 0 1, limit lower=-1.91986 upper=1.91986 effort=10 velocity=10
- added joint Wrist_Pitch: type revolute, parent lower_arm, child wrist, origin xyz=-0.1349 0.0052 1.65232e-16 rpy=3.2474e-15 2.86219e-15 -1.5708, axis 0 0 1, limit lower=-1.65806 upper=1.65806 effort=10 velocity=10
- added joint Wrist_Roll: type revolute, parent wrist, child gripper, origin xyz=0 -0.0611 0.0181 rpy=1.5708 -9.38083e-08 3.14159, axis 0 0 1, limit lower=-2.79253 upper=2.79253 effort=10 velocity=10
- joint world_to_base: axis 0 0 0 -> (none); child base_link -> base; origin xyz=0.0137179 -5.19711e-05 0.0334843 rpy=0.0 0.0 0.0 -> xyz=0 0 0 rpy=0 0 0

File: so101_description/urdf/so101_new_calib_with_transmission.xacro (robot description, xacro)
@@ -1,63 +1,63 @@
 <?xml version="1.0"?>
 <robot xmlns:xacro="http://ros.org/wiki/xacro" name="so101_new_calib">
-    <transmission name="6_trans">
+    <transmission name="gripper_trans">
         <type>transmission_interface/SimpleTransmission</type>
-        <joint name="Jaw">
-        <hardwareInterface>hardware_interface/PositionJointInterface</hardwareInterface>
+        <joint name="gripper">
+          <hardwareInterface>hardware_interface/PositionJointInterface</hardwareInterface>
         </joint>
         <actuator name="motor6">
-        <hardwareInterface>hardware_interface/PositionJointInterface</hardwareInterface>
-        <mechanicalReduction>1</mechanicalReduction>
+          <hardwareInterface>hardware_interface/PositionJointInterface</hardwareInterface>
+          <mechanicalReduction>1</mechanicalReduction>
         </actuator>
-    </transmission>
-    <transmission name="5_trans">
+      </transmission>
+    <transmission name="wrist_roll_trans">
         <type>transmission_interface/SimpleTransmission</type>
-        <joint name="Wrist_Roll">
-        <hardwareInterface>hardware_interface/PositionJointInterface</hardwareInterface>
+        <joint name="wrist_roll">
+          <hardwareInterface>hardware_interface/PositionJointInterface</hardwareInterface>
         </joint>
         <actuator name="motor5">
-        <hardwareInterface>hardware_interface/PositionJointInterface</hardwareInterface>
-        <mechanicalReduction>1</mechanicalReduction>
+          <hardwareInterface>hardware_interface/PositionJointInterface</hardwareInterface>
+          <mechanicalReduction>1</mechanicalReduction>
         </actuator>
-    </transmission>
-    <transmission name="4_trans">
+      </transmission>
+    <transmission name="wrist_flex_trans">
         <type>transmission_interface/SimpleTransmission</type>
-        <joint name="Wrist_Pitch">
-        <hardwareInterface>hardware_interface/PositionJointInterface</hardwareInterface>
+        <joint name="wrist_flex">
+          <hardwareInterface>hardware_interface/PositionJointInterface</hardwareInterface>
         </joint>
         <actuator name="motor4">
-        <hardwareInterface>hardware_interface/PositionJointInterface</hardwareInterface>
-        <mechanicalReduction>1</mechanicalReduction>
+          <hardwareInterface>hardware_interface/PositionJointInterface</hardwareInterface>
+          <mechanicalReduction>1</mechanicalReduction>
         </actuator>
-    </transmission>
-    <transmission name="3_trans">
+      </transmission>
+    <transmission name="elbow_flex_trans">
         <type>transmission_interface/SimpleTransmission</type>
-        <joint name="Elbow">
-        <hardwareInterface>hardware_interface/PositionJointInterface</hardwareInterface>
+        <joint name="elbow_flex">
+          <hardwareInterface>hardware_interface/PositionJointInterface</hardwareInterface>
         </joint>
         <actuator name="motor3">
-        <hardwareInterface>hardware_interface/PositionJointInterface</hardwareInterface>
-        <mechanicalReduction>1</mechanicalReduction>
+          <hardwareInterface>hardware_interface/PositionJointInterface</hardwareInterface>
+          <mechanicalReduction>1</mechanicalReduction>
         </actuator>
-    </transmission>
-    <transmission name="2_trans">
+      </transmission>
+    <transmission name="shoulder_lift_trans">
         <type>transmission_interface/SimpleTransmission</type>
-        <joint name="Pitch">
-        <hardwareInterface>hardware_interface/PositionJointInterface</hardwareInterface>
+        <joint name="shoulder_lift">
+          <hardwareInterface>hardware_interface/PositionJointInterface</hardwareInterface>
         </joint>
         <actuator name="motor2">
-        <hardwareInterface>hardware_interface/PositionJointInterface</hardwareInterface>
-        <mechanicalReduction>1</mechanicalReduction>
+          <hardwareInterface>hardware_interface/PositionJointInterface</hardwareInterface>
+          <mechanicalReduction>1</mechanicalReduction>
         </actuator>
-    </transmission>
-    <transmission name="1_trans">
+      </transmission>
+    <transmission name="shoulder_pan_trans">
         <type>transmission_interface/SimpleTransmission</type>
-        <joint name="Rotation">
-        <hardwareInterface>hardware_interface/PositionJointInterface</hardwareInterface>
+        <joint name="shoulder_pan">
+          <hardwareInterface>hardware_interface/PositionJointInterface</hardwareInterface>
         </joint>
         <actuator name="motor1">
-        <hardwareInterface>hardware_interface/PositionJointInterface</hardwareInterface>
-        <mechanicalReduction>1</mechanicalReduction>
+          <hardwareInterface>hardware_interface/PositionJointInterface</hardwareInterface>
+          <mechanicalReduction>1</mechanicalReduction>
         </actuator>
-    </transmission>
+      </transmission>
 </robot>
